File: Ivy Sensor.sch (EAGLE design)
At the start: 14 parts, among them SW1 OS102011MA1Q

Commit message: Update design to version 0.3
Parts:
- removed RSV: Reserved, SparkFun-Connectors:M03PTH
- added Q1: C1815, SparkFun-DiscreteSemi:TRANSISTOR_NPNSOT23-3
- added R1: 10K, resistor:R-US_R0805
Connections:
- new net N$1: BUZZER.2, Q1.C
- new net N$3: Q1.B, R1.1
- net 5V: now also BUZZER.1; no longer RSV.1
- net D2: now also SW1G$1.P; no longer DHT22.DATA, R4.2
- net D3: now also DHT22.DATA, R4.2; no longer RSV.2
- net D4: now also R1.2; no longer BUZZER.1
- net D6: no longer SW1G$1.P
- net GND: now also Q1.E; no longer BUZZER.2, RSV.3
Other:
- note added: "2016-10-13 http://easytech.vn"
- note added: "Ivy Home Sensor V0.3"
- note removed: "2016-10-05 http://easytech.vn"
- note removed: "Ivy Home Sensor V0.2"
- moved on the sheet: BUZZER

Commit message: Update design to version 0.4
Parts:
- removed Q1: C1815, SparkFun-DiscreteSemi:TRANSISTOR_NPNSOT23-3
- removed SW1: OS102011MA1Q, adafruit:OS102011MA1Q
- added BTN: OS102011MA1Q, adafruit:OS102011MA1Q
- added JP1, JP2: (no value), SparkFun-Connectors:M08
- added Q2: A1015, SparkFun-DiscreteSemi:TRANSISTOR_PNPSMD
- C1: value 47uF/16V -> 47uF
Connections:
- removed net N$1: BUZZER.2, Q1.C
- removed net N$3: Q1.B, R1.1
- new net RX: JP2.2, U$2.RX
- new net TX: JP2.1, U$2.TX
- new net T_B: Q2.B, R1.1
- new net T_C: BUZZER.1, Q2.C
- net 5V: now also JP2.8, Q2.E; no longer BUZZER.1
- net A0: now also JP1.7
- net D0: now also JP1.6
- net D1: now also JP2.3
- net D2: now also BTNG$1.P, JP2.4; no longer SW1G$1.P
- net D3: now also JP2.5
- net D4: now also JP2.6
- net D5: now also JP1.5
- net D6: now also JP1.4
- net D7: now also JP1.3
- net D8: now also JP1.2
- net GND: now also BTNG$1.S, BUZZER.2, JP2.7; no longer Q1.E, SW1G$1.S
- net RST: now also JP1.8
- net VCC: now also JP1.1; no longer SW1G$1.O
Other:
- note added: "2016-10-16 http://easytech.vn"
- note added: "Display & Inputs"
- note added: "Ivy Home Sensor V0.4"
- note removed: "2016-10-13 http://easytech.vn"
- note removed: "Display & Control"
- note removed: "Ivy Home Sensor V0.3"
- moved on the sheet: BATT, BUZZER, DEEP_SLEEP_JP, R1, U$2

Commit message: Update design to version 0.5
Parts:
- R1: value 10K -> 47K
Other:
- note added: "2016-10-24 http://easytech.vn"
- note added: "Ivy Home Sensor V0.5"
- note removed: "2016-10-16 http://easytech.vn"
- note removed: "Ivy Home Sensor V0.4"
Changed lines of the file:
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@@
 <part name="C2" library="SparkFun-Capacitors" deviceset="CAP_POL" device="PTH2" value="102pF"/>
 <part name="GND5" library="SparkFun" deviceset="GND" device=""/>
-<part name="R1" library="resistor" deviceset="R-US_" device="R0805" value="10K"/>
+<part name="R1" library="resistor" deviceset="R-US_" device="R0805" value="47K"/>
 <part name="Q2" library="SparkFun-DiscreteSemi" deviceset="TRANSISTOR_PNP" device="SMD" value="A1015"/>
 <part name="JP1" library="SparkFun-Connectors" deviceset="M08" device=""/>
@@
 <wire x1="304.8" y1="40.64" x2="137.16" y2="40.64" width="0.1524" layer="97"/>
 <wire x1="137.16" y1="40.64" x2="137.16" y2="91.44" width="0.1524" layer="97"/>
-<text x="238.76" y="81.28" size="3.81" layer="97" font="vector" ratio="15">Ivy Home Sensor V0.4</text>
-<text x="238.76" y="71.12" size="2.54" layer="97" font="vector" ratio="15">2016-10-16
+<text x="238.76" y="81.28" size="3.81" layer="97" font="vector" ratio="15">Ivy Home Sensor V0.5</text>
+<text x="238.76" y="71.12" size="2.54" layer="97" font="vector" ratio="15">2016-10-24
 http://easytech.vn</text>
 <wire x1="137.16" y1="38.1" x2="304.8" y2="38.1" width="0.1524" layer="97"/>

Commit message: Update design to version 1.0
Other:
- note added: "Ivy Home Sensor v1.0"
- note removed: "Ivy Home Sensor V0.5"
Changed lines of the file:
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@@
 <wire x1="304.8" y1="40.64" x2="137.16" y2="40.64" width="0.1524" layer="97"/>
 <wire x1="137.16" y1="40.64" x2="137.16" y2="91.44" width="0.1524" layer="97"/>
-<text x="238.76" y="81.28" size="3.81" layer="97" font="vector" ratio="15">Ivy Home Sensor V0.5</text>
-<text x="238.76" y="71.12" size="2.54" layer="97" font="vector" ratio="15">2016-10-24
+<text x="236.22" y="81.28" size="3.81" layer="97" font="vector" ratio="15">Ivy Home Sensor v1.0</text>
+<text x="236.22" y="71.12" size="2.54" layer="97" font="vector" ratio="15">2016-10-24
 http://easytech.vn</text>
 <wire x1="137.16" y1="38.1" x2="304.8" y2="38.1" width="0.1524" layer="97"/>
